File: pcb/BSV.kicad_pcb (KiCad board)
At the start: 2 copper layers, 87.6 x 53.3 mm, 54 parts, among them J1 Conn_01x02_Pin, J2 Conn_01x02_Pin, J3 Conn_01x02_Pin, J4 Conn_01x02_Socket, J5 Conn_01x03_Pin, J6 AudioJack3, Q1 BC337, Q2 BC337, Q3 BC327, Q4 BC327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

Commit message: Adapt PCB variables
Other:
- board text added: "${title}"
- board text added: "Creator: ${creator}"
- board text added: "Version: ${revision}"
- board text removed: "Creator: GAR"
- board text removed: "Stereoverstärker"
- board text removed: "Version: 2.0"
Changed lines of the file:
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@@
     (effects (font (size 1 1) (thickness 0.15)) (justify left bottom mirror))
   )
-  (gr_text "Stereoverstärker" (at 183.515 114.3) (layer "B.SilkS")
+  (gr_text "${title}" (at 183.515 114.3) (layer "B.SilkS")
     (effects (font (size 1 1) (thickness 0.15)) (justify left bottom mirror))
   )
-  (gr_text "Creator: GAR" (at 183.388 117.856) (layer "B.SilkS")
+  (gr_text "Creator: ${creator}" (at 183.388 117.856) (layer "B.SilkS")
     (effects (font (size 1 1) (thickness 0.15)) (justify left bottom mirror))
   )
@@
     (effects (font (size 1 1) (thickness 0.15)) (justify left bottom mirror))
   )
-  (gr_text "Version: 2.0" (at 183.388 116.078) (layer "B.SilkS")
+  (gr_text "Version: ${revision}" (at 183.388 116.078) (layer "B.SilkS")
     (effects (font (size 1 1) (thickness 0.15)) (justify left bottom mirror))
   )
